Commit message: randomized worlds, add contact sensor (not working when spawning the model through ros_gz and no ros bridge for the corresponding message, cant wait to stop using outdated tools)

File: resources/environment_assets/objects_large/unused/cube_1m.urdf (robot description, URDF)
Before this commit: robot box, 1 links, 0 joints
Links:
- link base_link: geometry collision box size=1.0 1.0 1.0; visual box size=1.0 1.0 1.0

File: resources/environment_assets/objects_large/unused/cuboidal_rod_1m.urdf (robot description, URDF)
Before this commit: robot box, 1 links, 0 joints
Links:
- link base_link: geometry collision box size=1 1 3.0; visual box size=1 1 3.0

File: resources/environment_assets/objects_large/unused/cuboidal_rod_60cm.urdf (robot description, URDF)
Before this commit: robot box, 1 links, 0 joints
Links:
- link base_link: geometry collision box size=0.6 0.6 3.0; visual box size=0.6 0.6 3.0

File: resources/environment_assets/objects_large/unused/sphere_1m.urdf (robot description, URDF)
Before this commit: robot box, 1 links, 0 joints
Links:
- link base_link: geometry collision sphere radius=1.0; visual sphere radius=1.0

File: resources/environment_assets/objects_medium/unused/cuboidal_rod_15cm.urdf (robot description, URDF)
Before this commit: robot box, 1 links, 0 joints
Links:
- link base_link: geometry collision box size=0.15 0.15 2.0; visual box size=0.15 0.15 2.0

File: resources/environment_assets/panels/unused/panel_1m.urdf (robot description, URDF)
Before this commit: robot box, 1 links, 0 joints
Links:
- link base_link: geometry collision box size=0.1 1.0 1.0; visual box size=0.1 1.0 1.0

File: resources/environment_assets/panels/unused/panel_2m.urdf (robot description, URDF)
Before this commit: robot box, 1 links, 0 joints
Links:
- link base_link: geometry collision box size=0.1 2.0 2.0; visual box size=0.1 2.0 2.0

File: resources/environment_assets/panels/unused/panel_50cm.urdf (robot description, URDF)
Before this commit: robot box, 1 links, 0 joints
Links:
- link base_link: geometry collision box size=0.1 0.5 0.5; visual box size=0.1 0.5 0.5

File: resources/environment_assets/pillars/unused/10cm_pillar.urdf (robot description, URDF)
Before this commit: robot pillar, 1 links, 0 joints
Links:
- link base_link: geometry collision cylinder length=8 radius=0.05; visual cylinder length=8 radius=0.05

File: resources/environment_assets/pillars/unused/10cm_pillar_rect.urdf (robot description, URDF)
Before this commit: robot pillar, 1 links, 0 joints
Links:
- link base_link: geometry collision box size=0.07 0.07 8; visual box size=0.07 0.07 8

File: resources/environment_assets/pillars/unused/1m_pillar.urdf (robot description, URDF)
Before this commit: robot pillar, 1 links, 0 joints
Links:
- link base_link: geometry collision cylinder length=8 radius=0.5; visual cylinder length=8 radius=0.5

File: resources/environment_assets/pillars/unused/20cm_pillar.urdf (robot description, URDF)
Before this commit: robot pillar, 1 links, 0 joints
Links:
- link base_link: geometry collision cylinder length=8 radius=0.1; visual cylinder length=8 radius=0.1

File: resources/environment_assets/pillars/unused/20cm_pillar_rect.urdf (robot description, URDF)
Before this commit: robot pillar, 1 links, 0 joints
Links:
- link base_link: geometry collision box size=0.14 0.14 8; visual box size=0.14 0.14 8

File: resources/environment_assets/pillars/unused/50cm_pillar.urdf (robot description, URDF)
Before this commit: robot pillar, 1 links, 0 joints
Links:
- link base_link: geometry collision cylinder length=8 radius=0.25; visual cylinder length=8 radius=0.25

File: resources/environment_assets/pillars/unused/5cm_pillar.urdf (robot description, URDF)
Before this commit: robot pillar, 1 links, 0 joints
Links:
- link base_link: geometry collision cylinder length=8 radius=0.025; visual cylinder length=8 radius=0.025

File: resources/environment_assets/thin/unused/cuboidal_rod_2cm.urdf (robot description, URDF)
Before this commit: robot box, 1 links, 0 joints
Links:
- link base_link: geometry collision box size=0.02 0.02 2.0; visual box size=0.02 0.02 2.0

File: resources/environment_assets/thin/unused/cuboidal_rod_5cm.urdf (robot description, URDF)
Before this commit: robot box, 1 links, 0 joints
Links:
- link base_link: geometry collision box size=0.05 0.05 2.0; visual box size=0.05 0.05 2.0

File: resources/environment_assets/thin/unused/cylinder_2cm.urdf (robot description, URDF)
Before this commit: robot box, 1 links, 0 joints
Links:
- link base_link: geometry collision cylinder length=2.0 radius=0.02; visual cylinder length=2.0 radius=0.02
